File: KiCad/arduino_pro_mini.kicad_sch (KiCad schematic)
At the start: 27 parts, among them IC101 UA78M05CDCYR, IC102 ATMEGA328P-AU, J101 Conn_01x06_Pin, J102 Conn_01x15_Pin, J103 Conn_01x15_Pin, J104 Conn_02x03_Odd_Even, SW101 SW_Omron_B3FS, Y101 16Mhz

Commit message: Update BOM
Parts:
- C101, C105, C106: Manufacturer Part Number (none) -> TAJA106K016RNJ; Manufacturer Product Number TAJA106K016RNJ -> (none)
- C102, C103, C104, C107, C110: Manufacturer Samsung Electro-Mechanics -> YAGEO; Manufacturer Part Number CL05B104KO5NNNC -> CC0805KRX7R9BB104
- C108, C109: Manufacturer Murata Electronics -> YAGEO; Manufacturer Part Number (none) -> CC0603JRNPO9BN150; Manufacturer Product Number GJM1555C1H150FB01D -> (none)
- IC101: Manufacturer (none) -> TI; Manufacturer Part Number (none) -> UA78M05CDCYR
- IC102: Manufacturer (none) -> MICROCHIP; Manufacturer Part Number (none) -> ATMEGA328P-AU; Manufacturer_Name Microchip -> (none); Manufacturer_Part_Number ATMEGA328P-AU -> (none); Mouser Part Number 556-ATMEGA328P-AU -> (none); Mouser Price/Stock https://www.mouser.co.uk/ProductDetail/Microchip-Technology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 -> (none)
- R101, R102, R103, R104, R105: Manufacturer (none) -> YAGEO; Manufacturer Part Number (none) -> RC0603FR-071KL
- SW101: Manufacturer Part Number (none) -> TSA063G50-250; Manufacturer Product Number TSA063G60-250 -> (none)
- Y101: Manufacturer Part Number (none) -> X322516MOB4SI; Manufacturer Product Number X322516MLB4SI -> (none)
Changed lines of the file:
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@@
 			)
 		)
-		(property "Manufacturer" "Samsung Electro-Mechanics"
+		(property "Manufacturer" "YAGEO"
 			(at 50.8 146.05 0)
 			(effects
@@
 			)
 		)
-		(property "Manufacturer Part Number" "CL05B104KO5NNNC"
-			(at 50.8 146.05 0)
-			(effects
-				(font
-					(size 1.27 1.27)
-				)
-				(hide yes)
-			)
-		)
-		(property "MANUFACTURER" ""
+		(property "Manufacturer Part Number" "CC0805KRX7R9BB104"
 			(at 50.8 146.05 0)
 			(effects
@@
 			)
 		)
-		(property "Manufacturer" ""
-			(at 107.95 82.55 0)
-			(effects
-				(font
-					(size 1.27 1.27)
-				)
-				(hide yes)
-			)
-		)
-		(property "Manufacturer Part Number" ""
+		(property "Manufacturer" "YAGEO"
 			(at 107.95 82.55 0)
 			(effects
@@
 			)
 		)
-		(property "MANUFACTURER" ""
+		(property "Manufacturer Part Number" "RC0603FR-071KL"
 			(at 107.95 82.55 0)
 			(effects
@@
 			)
 		)
-		(property "Manufacturer Product Number" "TSA063G60-250"
+		(property "Manufacturer Part Number" "TSA063G50-250"
 			(at 36.83 138.43 0)
 			(effects
@@
 			)
 		)
-		(property "Manufacturer" "Samsung Electro-Mechanics"
-			(at 184.15 35.56 0)
-			(effects
-				(font
-					(size 1.27 1.27)
-				)
-				(hide yes)
-			)
-		)
-		(property "Manufacturer Part Number" "CL05B104KO5NNNC"
+		(property "Manufacturer" "YAGEO"
 			(at 184.15 35.56 0)
 			(effects
@@
 			)
 		)
-		(property "MANUFACTURER" ""
+		(property "Manufacturer Part Number" "CC0805KRX7R9BB104"
 			(at 184.15 35.56 0)
 			(effects
@@
 			)
 		)
+		(property "Manufacturer" "TI"
+			(at 33.02 30.48 0)
+			(effects
+				(font
+					(size 1.27 1.27)
+				)
+				(hide yes)
+			)
+		)
+		(property "Manufacturer Part Number" "UA78M05CDCYR"
+			(at 33.02 30.48 0)
+			(effects
+				(font
+					(size 1.27 1.27)
+				)
+				(hide yes)
+			)
+		)
 		(pin "4"
 		)
@@
 			)
 		)
-		(property "Manufacturer" "Samsung Electro-Mechanics"
-			(at 166.37 35.56 0)
-			(effects
-				(font
-					(size 1.27 1.27)
-				)
-				(hide yes)
-			)
-		)
-		(property "Manufacturer Part Number" "CL05B104KO5NNNC"
+		(property "Manufacturer" "YAGEO"
 			(at 166.37 35.56 0)
 			(effects
@@
 			)
 		)
-		(property "MANUFACTURER" ""
+		(property "Manufacturer Part Number" "CC0805KRX7R9BB104"
 			(at 166.37 35.56 0)
 			(effects
@@
 			)
 		)
-		(property "Manufacturer" "Murata Electronics"
+		(property "Manufacturer" "YAGEO"
 			(at 25.4 90.17 0)
 			(effects
@@
 			)
 		)
-		(property "Manufacturer Product Number" "GJM1555C1H150FB01D"
+		(property "Manufacturer Part Number" "CC0603JRNPO9BN150"
 			(at 25.4 90.17 0)
 			(effects
@@
 			)
 		)
-		(property "Manufacturer Product Number" "TAJA106K016RNJ"
+		(property "Manufacturer Part Number" "TAJA106K016RNJ"
 			(at 21.59 39.37 0)
 			(effects
@@
 			)
 		)
-		(property "Manufacturer" "Murata Electronics"
+		(property "Manufacturer" "YAGEO"
 			(at 46.99 90.17 0)
 			(effects
@@
 			)
 		)
-		(property "Manufacturer Product Number" "GJM1555C1H150FB01D"
+		(property "Manufacturer Part Number" "CC0603JRNPO9BN150"
 			(at 46.99 90.17 0)
 			(effects
@@
 			)
 		)
-		(property "Manufacturer Product Number" "X322516MLB4SI"
+		(property "Manufacturer Part Number" "X322516MOB4SI"
 			(at 35.56 83.82 0)
 			(effects
@@
 			)
 		)
-		(property "Manufacturer" ""
-			(at 238.76 148.59 0)
-			(effects
-				(font
-					(size 1.27 1.27)
-				)
-				(hide yes)
-			)
-		)
-		(property "Manufacturer Part Number" ""
+		(property "Manufacturer" "YAGEO"
 			(at 238.76 148.59 0)
 			(effects
@@
 			)
 		)
-		(property "MANUFACTURER" ""
+		(property "Manufacturer Part Number" "RC0603FR-071KL"
 			(at 238.76 148.59 0)
 			(effects
@@
 			)
 		)
-		(property "Manufacturer Product Number" "TAJA106K016RNJ"
+		(property "Manufacturer Part Number" "TAJA106K016RNJ"
 			(at 54.61 39.37 0)
 			(effects
@@
 			)
 		)
-		(property "Manufacturer Product Number" "TAJA106K016RNJ"
+		(property "Manufacturer Part Number" "TAJA106K016RNJ"
 			(at 157.48 35.56 0)
 			(effects
@@
 			)
 		)
-		(property "Manufacturer" ""
-			(at 64.77 39.37 0)
-			(effects
-				(font
-					(size 1.27 1.27)
-				)
-				(hide yes)
-			)
-		)
-		(property "Manufacturer Part Number" ""
+		(property "Manufacturer" "YAGEO"
 			(at 64.77 39.37 0)
 			(effects
@@
 			)
 		)
-		(property "MANUFACTURER" ""
+		(property "Manufacturer Part Number" "RC0603FR-071KL"
 			(at 64.77 39.37 0)
 			(effects
@@
 			)
 		)
-		(property "Manufacturer" "Samsung Electro-Mechanics"
-			(at 175.26 35.56 0)
-			(effects
-				(font
-					(size 1.27 1.27)
-				)
-				(hide yes)
-			)
-		)
-		(property "Manufacturer Part Number" "CL05B104KO5NNNC"
+		(property "Manufacturer" "YAGEO"
 			(at 175.26 35.56 0)
 			(effects
@@
 			)
 		)
-		(property "MANUFACTURER" ""
+		(property "Manufacturer Part Number" "CC0805KRX7R9BB104"
 			(at 175.26 35.56 0)
 			(effects
@@
 			)
 		)
-		(property "Manufacturer" ""
+		(property "Manufacturer" "YAGEO"
 			(at 107.95 85.09 0)
 			(effects
@@
 			)
 		)
-		(property "Manufacturer Part Number" ""
-			(at 107.95 85.09 0)
-			(effects
-				(font
-					(size 1.27 1.27)
-				)
-				(hide yes)
-			)
-		)
-		(property "MANUFACTURER" ""
+		(property "Manufacturer Part Number" "RC0603FR-071KL"
 			(at 107.95 85.09 0)
 			(effects
@@
 			)
 		)
-		(property "Manufacturer_Name" "Microchip"
-			(at 245.11 517.78 0)
-			(effects
-				(font
-					(size 1.27 1.27)
-				)
-				(justify left top)
-				(hide yes)
-			)
-		)
-		(property "Manufacturer_Part_Number" "ATMEGA328P-AU"
-			(at 245.11 617.78 0)
-			(effects
-				(font
-					(size 1.27 1.27)
-				)
-				(justify left top)
-				(hide yes)
-			)
-		)
-		(property "Mouser Part Number" "556-ATMEGA328P-AU"
-			(at 245.11 717.78 0)
+		(property "Manufacturer" "MICROCHIP"
+			(at 177.8 53.34 0)
 			(effects
 				(font
 					(size 1.27 1.27)
 				)
-				(justify left top)
 				(hide yes)
 			)
 		)
-		(property "Mouser Price/Stock" "https://www.mouser.co.uk/ProductDetail/Microchip-Technology/ATMEGA328P-AU?qs=K8BHR703ZXiCmmgp6%2FGNmQ%3D%3D"
-			(at 245.11 817.78 0)
+		(property "Manufacturer Part Number" "ATMEGA328P-AU"
+			(at 177.8 53.34 0)
 			(effects
 				(font
 					(size 1.27 1.27)
 				)
-				(justify left top)
 				(hide yes)
 			)
@@
 			)
 		)
-		(property "Manufacturer" "Samsung Electro-Mechanics"
-			(at 167.64 63.5 0)
-			(effects
-				(font
-					(size 1.27 1.27)
-				)
-				(hide yes)
-			)
-		)
-		(property "Manufacturer Part Number" "CL05B104KO5NNNC"
+		(property "Manufacturer" "YAGEO"
 			(at 167.64 63.5 0)
 			(effects
@@
 			)
 		)
-		(property "MANUFACTURER" ""
+		(property "Manufacturer Part Number" "CC0805KRX7R9BB104"
 			(at 167.64 63.5 0)
 			(effects
@@
 			)
 		)
-		(property "Manufacturer" ""
-			(at 43.18 125.73 0)
-			(effects
-				(font
-					(size 1.27 1.27)
-				)
-				(hide yes)
-			)
-		)
-		(property "Manufacturer Part Number" ""
+		(property "Manufacturer" "YAGEO"
 			(at 43.18 125.73 0)
 			(effects
@@
 			)
 		)
-		(property "MANUFACTURER" ""
+		(property "Manufacturer Part Number" "RC0603FR-071KL"
 			(at 43.18 125.73 0)
 			(effects
